File: pcb/tram.stop.brd (EAGLE design)
At the start: 62.1 x 46.2 mm, 22 parts, among them Q1 BC847SMD, U1 ATTINY85V-10SU, U2 LM1117MP-5.0

Commit message: #! finalize code
Parts:
- removed JP4: (no value), pinhead:2X04/90
- removed JP5: (no value), pinhead:2X03/90
- removed JP6: (no value), pinhead:1X03/90
- removed JP7: (no value), pinhead:1X02/90
- added JP1: (no value), pinhead:1X07
- JP2: device pinhead:1X02/90 -> pinhead:1X06/90
- moved JP2 54.1 mm to (15.4, 52.8), turned to 90 degrees
- moved U1 0.38 mm to (53.5, 58.9)
- moved Q1 0.25 mm to (44.4, 53.2)
- moved U2 0.12 mm to (36.3, 59.1)
Connections:
- removed net N$1: JP2.1, U1.1
- new net N$13: JP1.6, JP2.6
- new net N$16: JP1.7, U1.1
- net JP1: now also JP2.1; no longer JP6.1
- net JP2: now also JP1.5, JP2.3; no longer JP5.1, JP5.2, JP6.3
- net N$10: now also JP1.3; no longer JP5.5, JP5.6
- net N$11: now also JP1.1; no longer JP7.2
- net N$12: now also JP2.4; no longer JP4.1, JP4.2
- net N$14: now also JP1.2; no longer JP7.1
- net N$15: now also JP1.4; no longer JP5.3, JP5.4
- net N$2: no longer JP2.2
- net N$21: now also JP2.2; no longer JP6.2
- net RED2: now also JP2.5; no longer JP4.3, JP4.4
Routing:
- net N$8: track 0.00 -> 39.4 mm
- net N$1: track 20.8 -> 0.00 mm
- net JP2: track 127.3 -> 123.0 mm
- net N$2: track 21.9 -> 18.6 mm
- net N$12: track 12.5 -> 10.4 mm
- net N$21: track 10.2 -> 8.05 mm
- net RED2: track 43.8 -> 41.7 mm
- net N$10: track 14.0 -> 12.3 mm
- net N$27: track 1.59 -> 0.00 mm
- net N$11: track 16.2 -> 14.7 mm
- net JP1: track 44.3 -> 42.9 mm
- net N$15: track 75.0 -> 73.7 mm
- net N$6: track 12.9 -> 11.8 mm
Other:
- board size 62.1 x 46.2 mm -> 52.3 x 24.5 mm
- board text added: "+ LED EOUT"
- board text removed: "+ R1 R2 WH"
